File: 8zu1AudioUmschalter.sch (KiCad schematic (older format))
At the start: 39 parts, among them IC1 ATMEGA8A-A, IC2 MAX9890, J1 USB, J2 LUM 1503-07, J3 LUM 1503-07, J4 LUM 1503-07, J5 LUM 1503-07, J6 LUM 1503-07, J7 LUM 1503-07, J8 LUM 1503-07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

Commit message: DTR nun als RESET für den Atmega Entfernen des Konnektors für ISP
Parts:
- removed P1: CONN_02X03, symbol CONN_02X03
- added C?: 100n, symbol C
Connections:
- net labels removed: /RESET, MISO, MOSI, SCK
- wire segments 149 -> 138
- no-connect marks 28 -> 31
Other:
- moved on the sheet: C10, C9
Changed lines of the file:
@@
 Entry Wire Line
 	6000 8150 6100 8050
-Entry Wire Line
-	6000 8300 6100 8200
 Wire Wire Line
 	6000 7700 5850 7700
@@
 Wire Wire Line
 	6000 8000 5850 8000
-Wire Wire Line
-	5850 8300 6000 8300
 Wire Wire Line
 	5850 8150 6000 8150
@@
 Text Label 5850 8300 0    60   ~ 0
 DTR
-Text Label 8250 5600 0    60   ~ 0
-DTR
-Entry Wire Line
-	8500 5600 8600 5500
-Wire Wire Line
-	8500 5600 8250 5600
 Text Label 8250 5500 0    60   ~ 0
 CTS
@@
 NoConn ~ 8250 5000
 $Comp
-L CONN_02X03 P1
-U 1 1 5504D8FC
-P 4900 6000
-F 0 "P1" H 4900 6200 50  0000 C CNN
-F 1 "CONN_02X03" H 4900 5800 50  0000 C CNN
-F 2 "" H 4900 4800 60  0000 C CNN
-F 3 "" H 4900 4800 60  0000 C CNN
-	1    4900 6000
-	1    0    0    -1
-$EndComp
-Wire Wire Line
-	5150 5900 5400 5900
-Wire Wire Line
-	5150 6000 5400 6000
-Wire Wire Line
-	5150 6100 5400 6100
-$Comp
-L GND #PWR011
-U 1 1 5504DE5D
-P 5400 6100
-F 0 "#PWR011" H 5400 5850 60  0001 C CNN
-F 1 "GND" H 5400 5950 60  0000 C CNN
-F 2 "" H 5400 6100 60  0000 C CNN
-F 3 "" H 5400 6100 60  0000 C CNN
-	1    5400 6100
-	1    0    0    -1
-$EndComp
-$Comp
-L VCC #PWR012
-U 1 1 5504DE89
-P 5400 5900
-F 0 "#PWR012" H 5400 5750 60  0001 C CNN
-F 1 "VCC" H 5400 6050 60  0000 C CNN
-F 2 "" H 5400 5900 60  0000 C CNN
-F 3 "" H 5400 5900 60  0000 C CNN
-	1    5400 5900
-	1    0    0    -1
-$EndComp
-Text Label 5200 6000 0    60   ~ 0
-MOSI
-Text Label 4350 5900 0    60   ~ 0
-MISO
-Text Label 4350 6000 0    60   ~ 0
-SCK
-Text Label 4300 6100 0    60   ~ 0
-/RESET
-Wire Wire Line
-	4650 5900 4250 5900
-Wire Wire Line
-	4250 6000 4650 6000
-Wire Wire Line
-	4650 6100 4250 6100
-$Comp
 L R R2
 U 1 1 5504E4FD
@@
 	6100 3300 6100 3200
 Wire Wire Line
-	5700 3600 6350 3600
+	6000 3600 6350 3600
 Connection ~ 6100 3600
-Text Label 5700 3600 0    60   ~ 0
-/RESET
-Text Label 8350 4100 0    60   ~ 0
-SCK
-Text Label 8350 4000 0    60   ~ 0
-MISO
-Text Label 8350 3900 0    60   ~ 0
-MOSI
-Wire Wire Line
-	8250 4100 8600 4100
-Wire Wire Line
-	8250 4000 8600 4000
-Wire Wire Line
-	8250 3900 8600 3900
 $Comp
 L C C6
@@
 $EndComp
 Wire Wire Line
-	5800 4000 5800 3900
+	5800 3900 5800 4000
 $Comp
 L GND #PWR015
@@
 L C C9
 U 1 1 5505028A
-P 7150 2950
-F 0 "C9" H 7175 3050 50  0000 L CNN
-F 1 "100n" H 7175 2850 50  0000 L CNN
-F 2 "" H 7188 2800 30  0000 C CNN
-F 3 "" H 7150 2950 60  0000 C CNN
-	1    7150 2950
-	1    0    0    -1
+P 7050 3200
+F 0 "C9" H 7075 3300 50  0000 L CNN
+F 1 "100n" H 7075 3100 50  0000 L CNN
+F 2 "" H 7088 3050 30  0000 C CNN
+F 3 "" H 7050 3200 60  0000 C CNN
+	1    7050 3200
+	0    -1   -1   0
 $EndComp
 $Comp
 L C C10
 U 1 1 55050318
-P 7350 2950
-F 0 "C10" H 7375 3050 50  0000 L CNN
-F 1 "100n" H 7375 2850 50  0000 L CNN
-F 2 "" H 7388 2800 30  0000 C CNN
-F 3 "" H 7350 2950 60  0000 C CNN
-	1    7350 2950
-	1    0    0    -1
-$EndComp
-Wire Wire Line
-	7300 3100 7300 3300
-Wire Wire Line
-	7200 3300 7200 3100
-Wire Wire Line
-	7150 3100 7350 3100
-Connection ~ 7300 3100
-Connection ~ 7200 3100
-Wire Wire Line
-	7150 2800 7350 2800
+P 7150 2900
+F 0 "C10" H 7175 3000 50  0000 L CNN
+F 1 "100n" H 7175 2800 50  0000 L CNN
+F 2 "" H 7188 2750 30  0000 C CNN
+F 3 "" H 7150 2900 60  0000 C CNN
+	1    7150 2900
+	0    -1   -1   0
+$EndComp
 $Comp
 L VCC #PWR018
 U 1 1 55050DE9
-P 7250 2800
-F 0 "#PWR018" H 7250 2650 60  0001 C CNN
-F 1 "VCC" H 7250 2950 60  0000 C CNN
-F 2 "" H 7250 2800 60  0000 C CNN
-F 3 "" H 7250 2800 60  0000 C CNN
-	1    7250 2800
+P 7300 2750
+F 0 "#PWR018" H 7300 2600 60  0001 C CNN
+F 1 "VCC" H 7300 2900 60  0000 C CNN
+F 2 "" H 7300 2750 60  0000 C CNN
+F 3 "" H 7300 2750 60  0000 C CNN
+	1    7300 2750
 	1    0    0    -1
 $EndComp
@@
 Wire Wire Line
 	6900 7200 6900 7150
-Wire Bus Line
-	6100 7550 6100 8300
-Wire Bus Line
-	6100 8300 6050 8300
 $Comp
 L JACK_2P J8
@@
 NoConn ~ 8250 3700
 NoConn ~ 8250 3600
+NoConn ~ 8250 4100
+NoConn ~ 8250 4000
+NoConn ~ 8250 3900
+$Comp
+L C C?
+U 1 1 5505E6C5
+P 5850 3600
+F 0 "C?" H 5875 3700 50  0000 L CNN
+F 1 "100n" H 5875 3500 50  0000 L CNN
+F 2 "" H 5888 3450 30  0000 C CNN
+F 3 "" H 5850 3600 60  0000 C CNN
+	1    5850 3600
+	0    1    1    0
+$EndComp
+Text Label 5450 3600 0    60   ~ 0
+DTR
+Wire Wire Line
+	5700 3600 5450 3600
+Wire Wire Line
+	7200 3200 7200 3300
+Wire Wire Line
+	7300 2750 7300 3300
+Wire Wire Line
+	7200 3200 7300 3200
+Connection ~ 7300 3200
+Connection ~ 7300 2900
+$Comp
+L GND #PWR?
+U 1 1 55060194
+P 6900 3200
+F 0 "#PWR?" H 6900 2950 60  0001 C CNN
+F 1 "GND" H 6900 3050 60  0000 C CNN
+F 2 "" H 6900 3200 60  0000 C CNN
+F 3 "" H 6900 3200 60  0000 C CNN
+	1    6900 3200
+	0    1    1    0
+$EndComp
+$Comp
+L GND #PWR?
+U 1 1 550601CF
+P 7000 2900
+F 0 "#PWR?" H 7000 2650 60  0001 C CNN
+F 1 "GND" H 7000 2750 60  0000 C CNN
+F 2 "" H 7000 2900 60  0000 C CNN
+F 3 "" H 7000 2900 60  0000 C CNN
+	1    7000 2900
+	0    1    1    0
+$EndComp
+Connection ~ 7200 3200
+Wire Bus Line
+	6100 7550 6100 8150
 $EndSCHEMATC
